Commit message: Fixed yumi model

File: yumi_srdf/srdf/yumi.srdf.xacro (robot description, xacro)
@@ -4,11 +4,6 @@
     A URDF file must exist for this robot as well, where the joints and the links that are referenced are defined
 -->
-<robot xmlns:xacro="http://ros.org/wiki/xacro" name="bigman">
+<robot xmlns:xacro="http://ros.org/wiki/xacro" name="yumi">
     <xacro:include filename="$(find yumi_urdf)/urdf/yumi_config.urdf.xacro" />
-    <virtual_joint name="virtual_joint" parent_frame="world" child_link="base_link" type="floating" />
-    <!--GROUPS: Representation of a set of joints and links. This can be useful for specifying DOF to plan for, defining arms, end effectors, etc-->
-    <!--LINKS: When a link is specified, the parent joint of that link (if it exists) is automatically included-->
-    <!--JOINTS: When a joint is specified, the child link of that joint (which will always exist) is automatically included-->
-    <!--CHAINS: When a chain is specified, all the links along the chain (including endpoints) are included in the group. Additionally, all the joints that are parents to included links are also included. This means that joints along the chain and the parent joint of the base link are included in the group-->
     <!--SUBGROUPS: Groups can also be formed by referencing to already defined group names-->
     <group name="base">
@@ -16,8 +11,8 @@
     </group>
     <group name="left_arm">
-        <chain base_link="yumi_link_1_l" tip_link="yumi_link_7_l"/>
+        <chain base_link="yumi_body" tip_link="yumi_link_7_l"/>
     </group>
     <group name="right_arm">
-        <chain base_link="yumi_link_1_r" tip_link="yumi_link_7_r"/>
+        <chain base_link="yumi_body" tip_link="yumi_link_7_r"/>
     </group>
     <!-- CONSTRAINT: first left then right -->

File: yumi_urdf/urdf/yumi.urdf.xacro (robot description, xacro)
@@ -10,7 +10,7 @@
   <xacro:include filename="$(find yumi_urdf)/urdf/yumi_fixed_gripper.xacro"/>
   <!-- Fix to world just for testing -->
-  <link name="world"/>
-  <xacro:yumi name="yumi" parent="world">
-    <origin xyz="0 0 0.1" rpy="0 0 0" />
+  <link name="base_link"/>
+  <xacro:yumi name="yumi" parent="base_link">
+    <origin xyz="0 0 0.0" rpy="0 0 0" />
   </xacro:yumi>
   <!--right gripper-->
